File: STM32H7B0_devboard/STM32H7B0_devboard.kicad_pcb (KiCad board)
At the start: 4 copper layers, 116.8 x 82.8 mm, 101 parts, among them J1 SWD, J2 24LC512 socet, J3 USB-C 16P, J4 PORT_A, J5 PORT_B, J6 PORT_C, J7 PORT_D, J8 PORT_E, J9 Power_Conn, Q1 S8050, Q2 AO3401A, SW1 BOOT_SEL, U1 STM32H7B0VBT6, U5 USBLC6-2SC6, Y1 32.768KHz, Y2 25MHz

Commit message: Constraints
Routing:
- net +3V3: track 34.4 -> 35.1 mm, vias 1 -> 2

Commit message: Layout V2
Parts:
- JP1, JP10, JP11, JP12, JP13, JP14, JP15, JP16, JP17, JP18, JP19, JP2, JP20, JP3, JP4, JP5, JP6, JP7, JP8, JP9, U2: moved to F.Cu
- moved H1 112.9 mm to (120.0, 40.0)
- moved H4 97.3 mm to (170.0, 120.0)
- moved J9 93.5 mm to (152.0, 40.0), turned to -90 degrees
- moved JP5 89.0 mm to (77.4, 61.5), turned to 0 degrees
- moved JP6 86.5 mm to (77.4, 65.0), turned to 0 degrees
- moved JP1 86.5 mm to (73.0, 61.5), turned to 0 degrees
- moved J4 86.5 mm to (136.9, 44.0), turned to 0 degrees
- moved J8 85.6 mm to (153.1, 44.0), turned to 0 degrees
- moved J5 85.6 mm to (141.0, 44.0), turned to 0 degrees
- moved J7 85.1 mm to (149.1, 44.0), turned to 0 degrees
- moved J6 85.1 mm to (145.0, 44.0), turned to 0 degrees
- moved JP10 84.2 mm to (81.7, 65.0), turned to 0 degrees
- moved JP2 81.8 mm to (73.0, 65.0), turned to 0 degrees
- moved J2 81.3 mm to (160.8, 51.4), turned to 0 degrees
- moved JP11 80.8 mm to (81.7, 68.6), turned to 0 degrees
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Connections:
- C18 pad 4: GND -> (no net)
Routing:
- net +5V: track 55.0 -> 14.9 mm
- net GND: track 79.7 -> 39.9 mm
- net /I2C_SDA: track 26.4 -> 0.00 mm, vias 1 -> 0
- net /I2C_SCL: track 25.2 -> 0.00 mm, vias 1 -> 0
- net /STATUS_LED: track 24.0 -> 0.00 mm, vias 2 -> 0
- net /BOOT0: track 0.00 -> 15.9 mm
- net +3V3: track 35.1 -> 22.2 mm, vias 2 -> 0
- net /power/BUCK_EN: track 12.2 -> 0.00 mm
- net /SWDIO: track 10.4 -> 0.00 mm, vias 1 -> 0
- net /power/BUCK_SW: track 9.59 -> 0.00 mm
- net Net-(D3-K): track 7.76 -> 0.00 mm
- net /HSE_IN: track 13.7 -> 6.48 mm
- net Net-(D3-A): track 5.98 -> 0.00 mm
- net /SWCLK: track 5.69 -> 0.00 mm, vias 1 -> 0
- net /LSE_IN: track 12.0 -> 6.45 mm
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Other:
- board outline removed
- board text removed: "${REFERENCE}"

Commit message: Buck
Parts:
- C14, C15, JP1, JP10, JP11, JP12, JP13, JP14, JP15, JP16, JP17, JP18, JP19, JP2, JP20, JP3, JP4, JP5, JP6, JP7, JP8, JP9, Q1, R12, R13, R14, R15, R16, R17, R18, U2: moved to B.Cu
- moved JP4 98.6 mm to (169.9, 90.6), turned to -90 degrees
- moved JP3 95.9 mm to (166.3, 90.6), turned to -90 degrees
- moved JP8 95.3 mm to (169.9, 95.0), turned to -90 degrees
- moved JP2 93.3 mm to (162.8, 90.6), turned to -90 degrees
- moved JP7 92.8 mm to (166.3, 95.0), turned to -90 degrees
- moved JP12 92.3 mm to (169.9, 99.3), turned to -90 degrees
- moved JP1 91.0 mm to (159.2, 90.6), turned to -90 degrees
- moved JP6 90.5 mm to (162.8, 95.0), turned to -90 degrees
- moved JP11 90.0 mm to (166.3, 99.3), turned to -90 degrees
- moved JP16 89.6 mm to (169.9, 103.7), turned to -90 degrees
- moved JP5 88.5 mm to (159.2, 95.0), turned to -90 degrees
- moved JP10 88.0 mm to (162.8, 99.3), turned to -90 degrees
- moved JP15 87.6 mm to (166.3, 103.7), turned to -90 degrees
- moved JP20 87.2 mm to (169.9, 108.0), turned to -90 degrees
- moved JP9 86.3 mm to (159.2, 99.3), turned to -90 degrees
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Connections:
- C18 pad 4: (no net) -> GND
Routing:
- net GND: track 39.9 -> 68.7 mm, vias 0 -> 7
- net +3V3: track 22.2 -> 39.2 mm, vias 0 -> 5
- net /power/BUCK_EN: track 0.00 -> 14.0 mm
- net /power/BUCK_FB: track 0.00 -> 10.9 mm
- net /power/BUCK_SW: track 0.00 -> 8.12 mm
- net +5V: track 14.9 -> 6.99 mm
- net Net-(D3-A): track 0.00 -> 4.61 mm
- net Net-(D3-K): track 0.00 -> 3.92 mm
- net Net-(Q2-D): track 0.00 -> 3.33 mm
- net /power/BUCK_BST: track 0.00 -> 2.64 mm
Other:
- board outline added: 60.4 x 90.4 mm
- board text added: "TODO ADD vias"

Commit message: Routing progress
Parts:
- moved Q1 68.4 mm to (164.4, 51.8), turned to 0 degrees
- moved U2 66.8 mm to (167.9, 57.6)
- moved J2 64.6 mm to (118.4, 100.2)
- moved R10 62.5 mm to (124.6, 112.2), turned to 180 degrees
- moved C14 62.0 mm to (165.8, 55.9), turned to -90 degrees
- moved R13 60.1 mm to (161.6, 51.0)
- moved R9 60.0 mm to (126.6, 112.2), turned to 0 degrees
- moved R14 59.7 mm to (161.6, 53.2)
- moved R12 58.8 mm to (165.3, 54.2), turned to 0 degrees
- moved C15 57.4 mm to (165.8, 64.4), turned to -90 degrees
- moved R18 53.4 mm to (164.9, 62.8), turned to 0 degrees
- moved R17 52.6 mm to (164.9, 61.6), turned to 180 degrees
- moved R15 50.5 mm to (164.9, 60.4), turned to 0 degrees
- moved R16 49.1 mm to (164.6, 64.4), turned to -90 degrees
- moved JP12 47.7 mm to (123.0, 107.8), turned to 180 degrees
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Routing:
- net GND: track 68.7 -> 131.2 mm, vias 7 -> 19
- net /A8: track 0.00 -> 40.0 mm
- net /A9: track 0.00 -> 38.0 mm
- net /A10: track 0.00 -> 35.2 mm
- net /QSPI1_NSS: track 2.18 -> 37.0 mm, vias 0 -> 2
- net /QSPI1_IO2: track 0.00 -> 34.0 mm, vias 0 -> 2
- net /QSPI1_IO1: track 0.00 -> 32.7 mm, vias 0 -> 2
- net /QSPI1_IO3: track 0.00 -> 31.5 mm, vias 0 -> 2
- net /QSPI1_SCK: track 0.00 -> 31.2 mm, vias 0 -> 2
- net /QSPI1_IO0: track 0.00 -> 30.0 mm, vias 0 -> 2
- net /A15: track 0.00 -> 29.9 mm, vias 0 -> 1
- net /I2C_SDA: track 0.00 -> 28.9 mm
- net Net-(J4-Pin_14): track 0.00 -> 28.3 mm
- net /I2C_SCL: track 0.00 -> 27.5 mm
- net Net-(J4-Pin_15): track 0.00 -> 27.3 mm
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- added copper zone on F.Cu, net +5V
Other:
- board text added: "TODO: More 3v3 and gnd vias for CPU"
- board text added: "TODO: USB wires PAIR!!"
- board text removed: "TODO ADD vias"

Commit message: Routing progress
Parts:
- moved JP13 18.2 mm to (161.2, 55.2), turned to 180 degrees
- moved JP18 11.9 mm to (161.2, 57.8), turned to 180 degrees
- moved JP15 10.0 mm to (161.2, 60.4), turned to 180 degrees
- moved JP16 9.82 mm to (161.2, 63.0), turned to 180 degrees
- moved JP14 7.60 mm to (161.2, 68.2), turned to 180 degrees
- moved JP11 5.05 mm to (128.0, 104.5), turned to 90 degrees
- moved JP12 3.54 mm to (124.0, 104.4), turned to 90 degrees
- moved JP17 2.47 mm to (161.2, 65.6), turned to 180 degrees
- moved C14 1.80 mm to (167.6, 55.9)
- moved C15 1.80 mm to (167.6, 64.4)
- moved Q1 1.80 mm to (166.2, 51.8)
- moved R15 1.80 mm to (166.7, 60.4)
- moved R17 1.80 mm to (166.7, 61.6)
- moved R18 1.80 mm to (166.7, 62.8)
- moved R12 1.80 mm to (167.1, 54.2)
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Connections:
- net /USB_DM renamed /USB_DN
- C18 pad 4: GND -> (no net)
Routing:
- net Net-(J5-Pin_12): track 0.00 -> 40.6 mm, vias 0 -> 1
- net Net-(J5-Pin_16): track 0.00 -> 33.7 mm, vias 0 -> 3
- net Net-(J5-Pin_15): track 0.00 -> 31.2 mm, vias 0 -> 1
- net Net-(J5-Pin_14): track 0.00 -> 30.0 mm, vias 0 -> 1
- net Net-(J5-Pin_13): track 0.00 -> 29.9 mm, vias 0 -> 1
- net Net-(J5-Pin_11): track 0.00 -> 29.6 mm, vias 0 -> 1
- net /A0: track 6.87 -> 32.2 mm
- net /D4: track 0.00 -> 24.2 mm
- net /C4: track 0.00 -> 24.2 mm
- net /B4: track 0.00 -> 24.1 mm
- net /A4: track 2.80 -> 26.2 mm
- net /A1: track 7.05 -> 30.3 mm
- net /USB_DN: track 3.98 -> 26.2 mm
- net /A5: track 2.50 -> 24.6 mm
- net /D5: track 0.00 -> 22.0 mm
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
Commit message: Routing process
Routing:
- net Net-(J4-Pin_7): track 20.2 -> 147.2 mm
- net /A2: track 26.0 -> 134.4 mm, vias 0 -> 1
- net /A5: track 24.6 -> 132.2 mm, vias 0 -> 1
- net /A4: track 26.2 -> 131.6 mm, vias 0 -> 1
- net /A3: track 24.7 -> 128.2 mm, vias 0 -> 1
- net /A1: track 30.3 -> 133.0 mm, vias 0 -> 1
- net /A0: track 32.2 -> 134.3 mm, vias 0 -> 1
- net Net-(J5-Pin_1): track 10.4 -> 110.1 mm, vias 0 -> 1
- net Net-(J4-Pin_8): track 23.6 -> 115.8 mm
- net Net-(J5-Pin_2): track 0.00 -> 86.7 mm, vias 0 -> 1
- net Net-(J5-Pin_3): track 0.00 -> 83.1 mm, vias 0 -> 1
- net Net-(J6-Pin_1): track 0.00 -> 71.7 mm, vias 0 -> 1
- net Net-(J5-Pin_4): track 0.00 -> 54.6 mm, vias 0 -> 1
- net Net-(J5-Pin_7): track 7.89 -> 53.1 mm, vias 0 -> 2
- net Net-(J5-Pin_8): track 8.28 -> 52.7 mm, vias 0 -> 1
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
Commit message: Routing done!
Parts:
- renumbered J4 to A, J5 to B, J6 to C, J7 to D, J8 to E, J9 to POWER
Connections:
- C18 pad 4: (no net) -> GND
Routing:
- net /E6: track 0.00 -> 120.4 mm, vias 0 -> 3
- net /E5: track 0.00 -> 117.2 mm, vias 0 -> 3
- net /E4: track 0.00 -> 113.9 mm, vias 0 -> 3
- net /E0: track 0.00 -> 101.2 mm, vias 0 -> 3
- net /E1: track 0.00 -> 101.2 mm, vias 0 -> 3
- net /E3: track 0.00 -> 101.1 mm, vias 0 -> 2
- net /E2: track 0.00 -> 100.4 mm, vias 0 -> 3
- net /D3: track 0.00 -> 93.1 mm, vias 0 -> 3
- net /D2: track 0.00 -> 89.4 mm, vias 0 -> 3
- net /D1: track 0.00 -> 86.1 mm, vias 0 -> 3
- net /D0: track 0.00 -> 82.1 mm, vias 0 -> 3
- net /D4: track 0.00 -> 71.0 mm, vias 0 -> 4
- net /D5: track 0.00 -> 66.8 mm, vias 0 -> 3
- net Net-(J8-Pin_12): track 0.00 -> 65.9 mm, vias 0 -> 2
- net /C1: track 4.42 -> 69.2 mm, vias 0 -> 1
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Other:
- board text added: "0"
- board text added: "15"
- board text removed: "TODO: More 3v3 and gnd vias for CPU"
- board text removed: "TODO: USB wires PAIR!!"

Commit message: Silk screen progress
Other:
- board text added: ","
