File: STM32H7B0_devboard/STM32H7B0_devboard.kicad_pcb (KiCad board)
At the start: 4 copper layers, 60.4 x 90.4 mm, 101 parts, among them J1 SWD, J2 24LC512 socet, J3 USB-C 16P, Q1 S8050, Q2 AO3401A, SW1 BOOT_SEL, U1 STM32H7B0VBT6, U5 USBLC6-2SC6, Y1 32.768KHz, Y2 25MHz

Commit message: Done V1
Other:
- outline, holes or cut-outs redrawn
- board text added: "1"
- board text added: "30"
- board text added: "JLCJLCJLCJLC"
- board text added: "No_0 05-2024"
- board text added: "STM32H7B0_devboard"

Commit message: Done V1.1
Parts:
- C14, C15, Q1, R12, R13, R14, R15, R16, R17, R18: moved to F.Cu
- renumbered A to J4, B to J5, C to J6, D to J7, E to J8, POWER to J9
Routing:
- net GND: track 144.9 -> 140.8 mm
- net /LCD_LEDK: track 5.52 -> 7.86 mm, vias 0 -> 1
- net /LCD_COMMAND: track 58.1 -> 60.4 mm
- net +3V3: track 75.0 -> 73.6 mm, vias 25 -> 24
- net /SPI2_NSS: track 46.6 -> 47.6 mm, vias 3 -> 4
- net /SPI2_SCK: track 57.0 -> 56.8 mm, vias 4 -> 3
- net /SPI2_MOSI: track 54.5 -> 54.3 mm, vias 4 -> 3
- net /LCD_RST: track 4.01 -> 4.18 mm, vias 0 -> 1
- net /LCD_NSS: vias 0 -> 1
- net /LCD_RESET: vias 1 -> 2

Commit message: Pin labels
Other:
- board text added: "00"
- board text added: "A"
- board text added: "B"
- board text added: "C"
- board text added: "D"
- board text added: "E"
- board text removed: "0"

Commit message: Manufacturer switch
Other:
- board text removed: "JLCJLCJLCJLC"
Changed lines of the file:
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@@
 		(tags "resistor")
 		(property "Reference" "R13"
-			(at 0 -1.62725 270)
+			(at 0 -1.62725 -90)
 			(layer "F.SilkS")
 			(effects
@@
 		)
 		(property "Value" "10k"
-			(at 0 1.17 270)
+			(at 0 1.17 -90)
 			(layer "F.Fab")
 			(effects
@@
 		)
 		(fp_text user "${REFERENCE}"
-			(at 0 0 270)
+			(at 0 0 -90)
 			(layer "F.Fab")
 			(effects
@@
 		(tags "SOT TO_SOT_SMD")
 		(property "Reference" "Q1"
-			(at -0.02725 -2.4 360)
+			(at -0.02725 -2.4 0)
 			(layer "F.SilkS")
 			(effects
@@
 		)
 		(property "Value" "S8050"
-			(at 0 2.4 360)
+			(at 0 2.4 0)
 			(layer "F.Fab")
 			(effects
@@
 		)
 		(fp_text user "${REFERENCE}"
-			(at 0 0 360)
+			(at 0 0 0)
 			(layer "F.Fab")
 			(effects
@@
 		(tags "resistor")
 		(property "Reference" "R12"
-			(at -1.937249 0 360)
+			(at -1.937249 0 0)
 			(layer "F.SilkS")
 			(effects
@@
 		)
 		(property "Value" "8r2"
-			(at 0 1.17 360)
+			(at 0 1.17 0)
 			(layer "F.Fab")
 			(effects
@@
 		)
 		(fp_text user "${REFERENCE}"
-			(at 0 0 360)
+			(at 0 0 0)
 			(layer "F.Fab")
 			(effects
@@
 		(tags "resistor")
 		(property "Reference" "R15"
-			(at 3.282749 0 360)
+			(at 3.282749 0 0)
 			(layer "F.SilkS")
 			(effects
@@
 		)
 		(property "Value" "2k2"
-			(at 0 1.17 360)
+			(at 0 1.17 0)
 			(layer "F.Fab")
 			(effects
@@
 		)
 		(fp_text user "${REFERENCE}"
-			(at 0 0 360)
+			(at 0 0 0)
 			(layer "F.Fab")
 			(effects
@@
 		(tags "resistor")
 		(property "Reference" "R14"
-			(at 0 -1.62725 270)
+			(at 0 -1.62725 -90)
 			(layer "F.SilkS")
 			(effects
@@
 		)
 		(property "Value" "1k"
-			(at 0 1.17 270)
+			(at 0 1.17 -90)
 			(layer "F.Fab")
 			(effects
@@
 		)
 		(fp_text user "${REFERENCE}"
-			(at 0 0 270)
+			(at 0 0 -90)
 			(layer "F.Fab")
 			(effects
@@
 		(at 169.7 57.65 90)
 		(property "Reference" "U2"
-			(at 0.05 3.7 270)
+			(at 0.05 3.7 -90)
 			(unlocked yes)
 			(layer "B.SilkS")
@@
 		)
 	)
-	(gr_text "JLCJLCJLCJLC\n"
-		(at 139.8 102 0)
-		(layer "F.SilkS")
-		(effects
-			(font
-				(size 1 1)
-				(thickness 0.1)
-			)
-			(justify left bottom)
-		)
-	)

Commit message: Finished board
Parts:
- removed SW1: BOOT_SEL, Button_Switch_SMD:Nidec_Copal_CAS-120A
- added JP21: ~, Jumper:SolderJumper-2_P1.3mm_Open_TrianglePad1.0x1.5mm, B.Cu at (135.0, 123.2)
- added JP22: ~, Jumper:SolderJumper-2_P1.3mm_Open_TrianglePad1.0x1.5mm, B.Cu at (135.0, 120.6)
- added R29: 10k, Resistor_SMD:R_0402_1005Metric, F.Cu at (138.0, 123.2)
Connections:
- C18 pad 4: GND -> (no net)
Routing:
- net GND: track 140.8 -> 136.9 mm
- net /BOOT0: track 15.9 -> 18.7 mm, vias 0 -> 1
- net Net-(JP21-B): track 0.00 -> 1.77 mm, vias 0 -> 1
- net +3V3: track 73.6 -> 72.7 mm
Other:
- board text added: "JLCJLCJLCJLC"

Commit message: Copper balance
Routing:
- net GND: vias 29 -> 84
- added copper zone on B.Cu, net GND
- added copper zone on F.Cu, net GND

Commit message: Copper balance
Routing:
- net GND: vias 84 -> 93
Changed lines of the file:
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@@
+	)
+	(via
+		(at 125.6 86)
+		(size 0.6)
+		(drill 0.3)
+		(layers "F.Cu" "B.Cu")
+		(free yes)
+		(net 2)
 	)
 	(via
@@
 	)
 	(via
-		(at 132 64)
+		(at 145.6 110.7)
 		(size 0.6)
 		(drill 0.3)
@@
 	)
 	(via
+		(at 117 80)
+		(size 0.6)
+		(drill 0.3)
+		(layers "F.Cu" "B.Cu")
+		(free yes)
+		(net 2)
+	)
+	(via
+		(at 122 91)
+		(size 0.6)
+		(drill 0.3)
+		(layers "F.Cu" "B.Cu")
+		(free yes)
+		(net 2)
+	)
+	(via
 		(at 158 94)
 		(size 0.6)
@@
 	)
 	(via
-		(at 171 83)
-		(size 0.6)
-		(drill 0.3)
-		(layers "F.Cu" "B.Cu")
-		(free yes)
-		(net 2)
-	)
-	(via
 		(at 169 85)
 		(size 0.6)
@@
 	)
 	(via
+		(at 150.4 45.1)
+		(size 0.6)
+		(drill 0.3)
+		(layers "F.Cu" "B.Cu")
+		(free yes)
+		(net 2)
+	)
+	(via
+		(at 122 86)
+		(size 0.6)
+		(drill 0.3)
+		(layers "F.Cu" "B.Cu")
+		(free yes)
+		(net 2)
+	)
+	(via
 		(at 130.5 85)
 		(size 0.6)
@@
 	)
 	(via
+		(at 139 49)
+		(size 0.6)
+		(drill 0.3)
+		(layers "F.Cu" "B.Cu")
+		(free yes)
+		(net 2)
+	)
+	(via
 		(at 154.211003 108.394579)
 		(size 0.6)
@@
 	)
 	(via
-		(at 132 62)
-		(size 0.6)
-		(drill 0.3)
-		(layers "F.Cu" "B.Cu")
-		(free yes)
-		(net 2)
-	)
-	(via
 		(at 168 78)
 		(size 0.6)
@@
 	)
 	(via
+		(at 127.2 98)
+		(size 0.6)
+		(drill 0.3)
+		(layers "F.Cu" "B.Cu")
+		(free yes)
+		(net 2)
+	)
+	(via
 		(at 148.017158 88.017158)
 		(size 0.6)
@@
 	)
 	(via
+		(at 149.7 96.2)
+		(size 0.6)
+		(drill 0.3)
+		(layers "F.Cu" "B.Cu")
+		(free yes)
+		(net 2)
+	)
+	(via
 		(at 144 106)
 		(size 0.6)
@@
 	)
 	(via
-		(at 132 68)
+		(at 130.8 72.1)
+		(size 0.6)
+		(drill 0.3)
+		(layers "F.Cu" "B.Cu")
+		(free yes)
+		(net 2)
+	)
+	(via
+		(at 150.4 49)
 		(size 0.6)
 		(drill 0.3)
@@
 	)
 	(via
+		(at 139 44)
+		(size 0.6)
+		(drill 0.3)
+		(layers "F.Cu" "B.Cu")
+		(free yes)
+		(net 2)
+	)
+	(via
 		(at 143 49)
 		(size 0.6)
 		(drill 0.3)
+		(layers "F.Cu" "B.Cu")
+		(free yes)
+		(net 2)
+	)
+	(via
+		(at 143.2 44)
+		(size 0.6)
+		(drill 0.3)
