File: STM32H7B0_devboard/STM32H7B0_devboard.kicad_sch (KiCad schematic)
At the start: 51 parts, among them J1 SWD, J2 24LC512 socet, Q2 S8050, SW1 BOOT_SEL, U1 STM32H7B0VBT6, Y1 25MHz, Y2 32.768KHz

Commit message: Breakout
Parts:
- added J4: PORT_A, Connector_PinSocket_2.00mm:PinSocket_1x16_P2.00mm_Vertical, symbol Connector_Generic:Conn_01x16
- added J5: PORT_B, Connector_PinSocket_2.00mm:PinSocket_1x16_P2.00mm_Vertical, symbol Connector_Generic:Conn_01x16
- added J6: PORT_C, Connector_PinSocket_2.00mm:PinSocket_1x16_P2.00mm_Vertical, symbol Connector_Generic:Conn_01x16
- added J7: PORT_D, Connector_PinSocket_2.00mm:PinSocket_1x16_P2.00mm_Vertical, symbol Connector_Generic:Conn_01x16
- added J8: PORT_E, Connector_PinSocket_2.00mm:PinSocket_1x16_P2.00mm_Vertical, symbol Connector_Generic:Conn_01x16
- added J9: Power_Conn, Connector_PinSocket_2.00mm:PinSocket_2x08_P2.00mm_Vertical, symbol Connector_Generic:Conn_02x08_Row_Letter_First
- added JP1, JP10, JP11, JP12, JP13, JP14, JP15, JP16, JP17, JP18, JP19, JP2, JP20, JP3, JP4, JP5, JP6, JP7, JP8, JP9: ~, symbol Jumper:SolderJumper_2_Open
- added R23, R24, R25, R26, R27, R28: 0, symbol Device:R_Small
- C12: renamed from C2; footprint (none) -> Capacitor_SMD:C_0402_1005Metric
- C13: renamed from C1; footprint (none) -> Capacitor_SMD:C_0402_1005Metric
- J1: footprint (none) -> Connector_PinSocket_2.00mm:PinSocket_2x05_P2.00mm_Vertical
- renumbered C3 to C1, C14 to C10, C15 to C11, C21 to C14, C20 to C15, C10 to C16, C11 to C17, C4 to C2, C5 to C3, C6 to C4, C7 to C5, C8 to C6, C9 to C7, C13 to C8, C12 to C9, D2 to D1, D1 to D2, Q2 to Q1, R8 to R1, R14 to R10, R22 to R11, R25 to R12, R26 to R13, R27 to R14, R24 to R15, R23 to R16, R29 to R17, R28 to R18, R9 to R5, R10 to R6, R11 to R7, R12 to R8, R13 to R9, U5 to U2, U4 to U3, Y2 to Y1, Y1 to Y2
Connections:
- net +3V3: now also J9.b1 (Pin_b1), J9.b2 (Pin_b2), J9.b3 (Pin_b3), J9.b4 (Pin_b4)
- net +5V: now also J9.b5 (Pin_b5), J9.b6 (Pin_b6), J9.b7 (Pin_b7), J9.b8 (Pin_b8)
- net GND: now also J9.a1 (Pin_a1), J9.a2 (Pin_a2), J9.a3 (Pin_a3), J9.a4 (Pin_a4), J9.a5 (Pin_a5), J9.a6 (Pin_a6), J9.a7 (Pin_a7), J9.a8 (Pin_a8)
- net I2C_SCL: now also JP11.1 (A)
- net I2C_SDA: now also JP12.1 (A)
- net LCD_BACKLIGHT: now also JP13.1 (A)
- net LCD_COMMAND: now also JP17.1 (A)
- net LCD_RESET: now also JP14.1 (A)
- net QSPI1_IO0: now also JP8.1 (A), R28.2; no longer U3.5 (D-DQ0)
- net QSPI1_IO1: now also JP7.1 (A), R24.1; no longer U3.2 (Q-DQ1)
- net QSPI1_IO2: now also JP2.1 (A), R25.1; no longer U3.3 (NW-DQ2)
- net QSPI1_IO3: now also JP1.1 (A), R26.2; no longer U3.7 (NH_DQ3)
- net QSPI1_NSS: now also JP20.1 (A), R23.1; no longer R11.1, U3.1 (NCS)
- net QSPI1_SCK: now also JP9.1 (A), R27.2; no longer U3.6 (CLK)
- net SPI2_MOSI: now also JP18.1 (A)
- net SPI2_NSS: now also JP15.1 (A)
- net SPI2_SCK: now also JP16.1 (A)
- net STATUS_LED: now also JP19.1 (A)
- net SWCLK: now also JP6.1 (A)
- net SWDIO: now also JP5.1 (A)
- net SWO: now also JP10.1 (A)
- net USB_DM: now also JP3.1 (A)
- net USB_DP: now also JP4.1 (A)
- net E2: now reaches U1.1 (PE2)
- net E2: now also J8.3 (Pin_3)
- net C1: now reaches U1.16 (PC1)
- net C1: now also J6.2 (Pin_2)
- net C2_C: now reaches U1.17 (PC2_C)
- net C2_C: now also J6.3 (Pin_3)
- net C3_C: now reaches U1.18 (PC3_C)
- net C3_C: now also J6.4 (Pin_4)
- net E3: now reaches U1.2 (PE3)
- net E3: now also J8.4 (Pin_4)
- net A0: now reaches U1.22 (PA0)
- net A0: now also U1.77 (PA15), J4.1 (Pin_1)
- net A1: now reaches U1.23 (PA1)
- net A1: now also J4.2 (Pin_2)
- net A2: now reaches U1.24 (PA2)
- net A2: now also J4.3 (Pin_3)
- net A3: now reaches U1.25 (PA3)
- net A3: now also J4.4 (Pin_4)
- net A4: now reaches U1.28 (PA4)
- net A4: now also J4.5 (Pin_5)
- net A5: now reaches U1.29 (PA5)
- net A5: now also J4.6 (Pin_6)
- net E4: now reaches U1.3 (PE4)
- net E4: now also J8.5 (Pin_5)
- net C4: now reaches U1.32 (PC4)
- net C4: now also J6.5 (Pin_5)
- net C5: now reaches U1.33 (PC5)
- net C5: now also J6.6 (Pin_6)
- net E7: now reaches U1.37 (PE7)
- net E7: now also J8.8 (Pin_8)
- net E8: now reaches U1.38 (PE8)
- net E8: now also J8.9 (Pin_9)
- net E9: now reaches U1.39 (PE9)
- net E9: now also J8.10 (Pin_10)
- net E5: now reaches U1.4 (PE5)
- net E5: now also J8.6 (Pin_6)
- net E10: now reaches U1.40 (PE10)
- net E10: now also J8.11 (Pin_11)
- net E12: now reaches U1.42 (PE12)
- net E12: now also J8.13 (Pin_13)
- net E13: now reaches U1.43 (PE13)
- net E13: now also J8.14 (Pin_14)
- net E14: now reaches U1.44 (PE14)
- net E14: now also J8.15 (Pin_15)
- net E15: now reaches U1.45 (PE15)
- net E15: now also J8.16 (Pin_16)
- net E6: now reaches U1.5 (PE6)
- net E6: now also J8.7 (Pin_7)
- net D8: now reaches U1.55 (PD8)
- net D8: now also J7.9 (Pin_9)
- net D9: now reaches U1.56 (PD9)
- net D9: now also J7.10 (Pin_10)
- net D10: now reaches U1.57 (PD10)
- net D10: now also J7.11 (Pin_11)
- net D11: now reaches U1.58 (PD11)
- net D11: now also J7.12 (Pin_12)
- net D12: now reaches U1.59 (PD12)
- net D12: now also J7.13 (Pin_13)
- net D13: now reaches U1.60 (PD13)
- net D13: now also J7.14 (Pin_14)
- net D14: now reaches U1.61 (PD14)
- net D14: now also J7.15 (Pin_15)
- net D15: now reaches U1.62 (PD15)
- net D15: now also J7.16 (Pin_16)
- net C6: now reaches U1.63 (PC6)
- net C6: now also J6.7 (Pin_7)
- net C7: now reaches U1.64 (PC7)
- net C7: now also J6.8 (Pin_8)
- net C8: now reaches U1.65 (PC8)
- net C8: now also J6.9 (Pin_9)
- net C9: now reaches U1.66 (PC9)
- net C9: now also J6.10 (Pin_10)
- net A8: now reaches U1.67 (PA8)
- net A8: now also J4.9 (Pin_9)
- net A9: now reaches U1.68 (PA9)
- net A9: now also J4.10 (Pin_10)
- net A10: now reaches U1.69 (PA10)
- net A10: now also J4.11 (Pin_11)
- net C13: now reaches U1.7 (PC13)
- net C13: now also J6.14 (Pin_14)
- net C10: now reaches U1.78 (PC10)
- net C10: now also J6.11 (Pin_11)
- net C11: now reaches U1.79 (PC11)
- net C11: now also J6.12 (Pin_12)
- net C12: now reaches U1.80 (PC12)
- net C12: now also J6.13 (Pin_13)
- net D0: now reaches U1.81 (PD0)
- net D0: now also J7.1 (Pin_1)
- net D1: now reaches U1.82 (PD1)
- net D1: now also J7.2 (Pin_2)
- net D2: now reaches U1.83 (PD2)
- net D2: now also J7.3 (Pin_3)
- net D3: now reaches U1.84 (PD3)
- net D3: now also J7.4 (Pin_4)
- net D4: now reaches U1.85 (PD4)
- net D4: now also J7.5 (Pin_5)
- net D5: now reaches U1.86 (PD5)
- net D5: now also J7.6 (Pin_6)
- net D6: now reaches U1.87 (PD6)
- net D6: now also J7.7 (Pin_7)
- net D7: now reaches U1.88 (PD7)
- net D7: now also J7.8 (Pin_8)
- net B4: now reaches U1.90 (PB4)
- net B4: now also J5.5 (Pin_5)
- net B5: now reaches U1.91 (PB5)
- net B5: now also J5.6 (Pin_6)
- net B8: now reaches U1.95 (PB8)
- net B8: now also J5.9 (Pin_9)
- net B9: now reaches U1.96 (PB9)
- net B9: now also J5.10 (Pin_10)
- net E0: now reaches U1.97 (PE0)
- net E0: now also J8.1 (Pin_1)
- net E1: now reaches U1.98 (PE1)
- net E1: now also J8.2 (Pin_2)
- new net: R28.1, U3.5 (D-DQ0)
- new net: J5.3 (Pin_3), JP9.2 (B)
- new net: J4.14 (Pin_14), JP5.2 (B)
- new net: J5.14 (Pin_14), JP16.2 (B)
- new net: J5.8 (Pin_8), JP12.2 (B)
- new net: J6.1 (Pin_1), JP19.2 (B)
- new net: J5.11 (Pin_11), JP13.2 (B)
- new net: J4.8 (Pin_8), JP2.2 (B)
- new net: J5.1 (Pin_1), JP7.2 (B)
- new net: J5.12 (Pin_12), JP14.2 (B)
- new net: J5.13 (Pin_13), JP15.2 (B)
- new net: J5.15 (Pin_15), JP17.2 (B)
- new net: J5.16 (Pin_16), JP18.2 (B)
- new net: J5.2 (Pin_2), JP8.2 (B)
- new net: J5.4 (Pin_4), JP10.2 (B)
- new net: J5.7 (Pin_7), JP11.2 (B)
- new net: J4.12 (Pin_12), JP3.2 (B)
- new net: J4.13 (Pin_13), JP4.2 (B)
- new net: R27.1, U3.6 (CLK)
- new net: R11.1, R23.2, U3.1 (NCS)
- new net: J4.7 (Pin_7), JP1.2 (B)
- new net: R25.2, U3.3 (NW-DQ2)
- new net: J8.12 (Pin_12), JP20.2 (B)
- new net: R24.2, U3.2 (Q-DQ1)
- new net: J4.15 (Pin_15), JP6.2 (B)
- new net: R26.1, U3.7 (NH_DQ3)
- new net A15: J4.16 (Pin_16)
- no-connect marks 66 -> 10
Other:
- note added: "Added zero-ohm bridges because QSPI code is still in testing"
- note added: "Breakout"
- note removed: "TODO low ESR!!"
- moved on the sheet: U3

Commit message: Schematic V2.0 + Footprints
Parts:
- J2: footprint (none) -> Package_DIP:CERDIP-8_W7.62mm_SideBrazed_Socket
- JP1, JP10, JP11, JP12, JP13, JP14, JP15, JP16, JP17, JP18, JP19, JP2, JP20, JP3, JP4, JP5, JP6, JP7, JP8, JP9: footprint (none) -> Jumper:SolderJumper-2_P1.3mm_Open_TrianglePad1.0x1.5mm
- L1: footprint (none) -> Inductor_SMD:L_0603_1608Metric
- R1, R10, R11, R12, R13, R14, R15, R16, R17, R18, R2, R3, R4, R5, R6, R7, R8, R9: footprint (none) -> Resistor_SMD:R_0402_1005Metric
- R23, R24, R25, R26, R27, R28: footprint (none) -> Resistor_SMD:R_0603_1608Metric
- U2: footprint (none) -> Custom:FPC_30_soldered
- U3: footprint (none) -> Package_SO:PowerIntegrations_SO-8
- Y1: footprint (none) -> Crystal:Crystal_SMD_3215-2Pin_3.2x1.5mm
- Y2: footprint (none) -> Crystal:Crystal_SMD_3225-4Pin_3.2x2.5mm
Other:
- note removed: "TODO: oscilator instead of Crystal (more precise and lower power!)"
Changed lines of the file:
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@@
 		)
 	)
-	(text "TODO:\noscilator instead of Crystal (more precise and lower power!)"
-		(exclude_from_sim no)
-		(at 173.228 56.134 0)
-		(effects
-			(font
-				(size 1.27 1.27)
-			)
-		)
-	)
 	(text "LCD"
 		(exclude_from_sim no)
@@
 			)
 		)
-		(property "Footprint" ""
+		(property "Footprint" "Resistor_SMD:R_0603_1608Metric"
 			(at 68.58 223.52 0)
 			(effects
@@
 			)
 		)
-		(property "Description" "Resistor, small symbol"
+		(property "Description" "0603WAF0000T5E"
 			(at 68.58 223.52 0)
 			(effects
@@
 			)
 		)
-		(property "Footprint" ""
+		(property "Footprint" "Jumper:SolderJumper-2_P1.3mm_Open_TrianglePad1.0x1.5mm"
 			(at 231.14 72.39 0)
 			(effects
@@
 			)
 		)
-		(property "Footprint" ""
+		(property "Footprint" "Jumper:SolderJumper-2_P1.3mm_Open_TrianglePad1.0x1.5mm"
 			(at 231.14 52.07 0)
 			(effects
@@
 			)
 		)
-		(property "Footprint" ""
+		(property "Footprint" "Resistor_SMD:R_0402_1005Metric"
 			(at 189.23 129.54 0)
 			(effects
@@
 			)
 		)
-		(property "Footprint" ""
+		(property "Footprint" "Jumper:SolderJumper-2_P1.3mm_Open_TrianglePad1.0x1.5mm"
 			(at 231.14 100.33 0)
 			(effects
@@
 			)
 		)
-		(property "Footprint" ""
+		(property "Footprint" "Resistor_SMD:R_0402_1005Metric"
 			(at 34.29 274.32 0)
 			(effects
@@
 			)
 		)
-		(property "Footprint" ""
+		(property "Footprint" "Resistor_SMD:R_0402_1005Metric"
 			(at 49.53 274.32 0)
 			(effects
@@
 			)
 		)
-		(property "Footprint" ""
+		(property "Footprint" "Jumper:SolderJumper-2_P1.3mm_Open_TrianglePad1.0x1.5mm"
 			(at 231.14 85.09 0)
 			(effects
@@
 			)
 		)
-		(property "Footprint" ""
+		(property "Footprint" "Resistor_SMD:R_0402_1005Metric"
 			(at 66.04 245.11 0)
 			(effects
@@
 			)
 		)
-		(property "Footprint" ""
+		(property "Footprint" "Package_DIP:CERDIP-8_W7.62mm_SideBrazed_Socket"
 			(at 168.91 180.34 0)
 			(effects
@@
 			)
 		)
-		(property "Footprint" ""
+		(property "Footprint" "Jumper:SolderJumper-2_P1.3mm_Open_TrianglePad1.0x1.5mm"
 			(at 231.14 92.71 0)
 			(effects
@@
 			)
 		)
-		(property "Footprint" ""
+		(property "Footprint" "Resistor_SMD:R_0402_1005Metric"
 			(at 151.13 163.83 0)
 			(effects
@@
 			)
 		)
-		(property "Footprint" ""
+		(property "Footprint" "Jumper:SolderJumper-2_P1.3mm_Open_TrianglePad1.0x1.5mm"
 			(at 231.14 36.83 0)
 			(effects
@@
 			)
 		)
-		(property "Footprint" ""
+		(property "Footprint" "Custom:FPC_30_soldered"
 			(at 121.92 200.66 0)
 			(effects
@@
 			)
 		)
-		(property "Footprint" ""
+		(property "Footprint" "Inductor_SMD:L_0603_1608Metric"
 			(at 152.4 265.43 0)
 			(effects
@@
 			)
 		)
-		(property "Description" "Inductor, small symbol"
+		(property "Description" "SDCL1608C39NJTDF"
 			(at 152.4 265.43 0)
 			(effects
@@
 			)
 		)
-		(property "Footprint" ""
+		(property "Footprint" "Resistor_SMD:R_0402_1005Metric"
 			(at 167.64 68.58 0)
 			(effects
@@
 			)
 		)
-		(property "Footprint" ""
+		(property "Footprint" "Jumper:SolderJumper-2_P1.3mm_Open_TrianglePad1.0x1.5mm"
 			(at 231.14 46.99 0)
 			(effects
@@
 			)
 		)
-		(property "Footprint" ""
+		(property "Footprint" "Resistor_SMD:R_0402_1005Metric"
 			(at 45.72 269.24 0)
 			(effects
@@
 			)
 		)
-		(property "Footprint" ""
+		(property "Footprint" "Resistor_SMD:R_0402_1005Metric"
 			(at 59.69 250.19 0)
 			(effects
@@
 			)
 		)
-		(property "Footprint" ""
+		(property "Footprint" "Resistor_SMD:R_0402_1005Metric"
 			(at 189.23 120.65 0)
 			(effects
@@
 			)
 		)
-		(property "Footprint" ""
+		(property "Footprint" "Jumper:SolderJumper-2_P1.3mm_Open_TrianglePad1.0x1.5mm"
 			(at 231.14 49.53 0)
 			(effects
@@
 			)
 		)
-		(property "Footprint" ""
+		(property "Footprint" "Resistor_SMD:R_0402_1005Metric"
 			(at 160.02 39.37 0)
 			(effects
@@
 			)
 		)
-		(property "Footprint" ""
+		(property "Footprint" "Resistor_SMD:R_0603_1608Metric"
 			(at 68.58 219.71 0)
 			(effects
@@
 			)
 		)
-		(property "Description" "Resistor, small symbol"
+		(property "Description" "0603WAF0000T5E"
 			(at 68.58 219.71 0)
 			(effects
@@
 			)
 		)
-		(property "Footprint" ""
+		(property "Footprint" "Resistor_SMD:R_0402_1005Metric"
 			(at 38.1 208.28 0)
 			(effects
@@
 			)
 		)
-		(property "Footprint" ""
+		(property "Footprint" "Crystal:Crystal_SMD_3225-4Pin_3.2x2.5mm"
 			(at 157.48 73.66 0)
 			(effects
@@
 			)
 		)
-		(property "Datasheet" "~"
+		(property "Datasheet" "https://www.lcsc.com/datasheet/lcsc_datasheet_2403291504_YXC-X322525MSB4SI_C13740.pdf"
 			(at 157.48 73.66 0)
 			(effects
@@
 			)
 		)
-		(property "Description" "Four pin crystal, GND on pins 2 and 4"
+		(property "Description" "X322525MSB4SI"
 			(at 157.48 73.66 0)
 			(effects
@@
 			)
 		)
-		(property "Footprint" ""
+		(property "Footprint" "Jumper:SolderJumper-2_P1.3mm_Open_TrianglePad1.0x1.5mm"
 			(at 231.14 34.29 0)
 			(effects
@@
 			)
 		)
-		(property "Footprint" ""
+		(property "Footprint" "Jumper:SolderJumper-2_P1.3mm_Open_TrianglePad1.0x1.5mm"
 			(at 231.14 67.31 0)
 			(effects
@@
 			)
 		)
-		(property "Footprint" ""
+		(property "Footprint" "Jumper:SolderJumper-2_P1.3mm_Open_TrianglePad1.0x1.5mm"
 			(at 231.14 82.55 0)
 			(effects
@@
 			)
 		)
-		(property "Footprint" ""
+		(property "Footprint" "Resistor_SMD:R_0402_1005Metric"
 			(at 189.23 138.43 0)
 			(effects
@@
 			)
 		)
-		(property "Footprint" ""
+		(property "Footprint" "Resistor_SMD:R_0603_1608Metric"
 			(at 33.02 219.71 0)
 			(effects
@@
 			)
 		)
-		(property "Description" "Resistor, small symbol"
+		(property "Description" "0603WAF0000T5E"
 			(at 33.02 219.71 0)
 			(effects
@@
 			)
 		)
-		(property "Footprint" ""
+		(property "Footprint" "Resistor_SMD:R_0402_1005Metric"
 			(at 189.23 147.32 0)
 			(effects
@@
 			)
 		)
-		(property "Footprint" ""
+		(property "Footprint" "Jumper:SolderJumper-2_P1.3mm_Open_TrianglePad1.0x1.5mm"
 			(at 231.14 102.87 0)
 			(effects
@@
 			)
 		)
-		(property "Footprint" ""
+		(property "Footprint" "Resistor_SMD:R_0402_1005Metric"
 			(at 83.82 242.57 0)
 			(effects
@@
 			)
 		)
-		(property "Footprint" ""
+		(property "Footprint" "Jumper:SolderJumper-2_P1.3mm_Open_TrianglePad1.0x1.5mm"
 			(at 231.14 97.79 0)
 			(effects
@@
 			)
 		)
-		(property "Footprint" ""
+		(property "Footprint" "Jumper:SolderJumper-2_P1.3mm_Open_TrianglePad1.0x1.5mm"
 			(at 231.14 95.25 0)
 			(effects
@@
 			)
 		)
-		(property "Footprint" ""
+		(property "Footprint" "Resistor_SMD:R_0603_1608Metric"
 			(at 33.02 215.9 0)
 			(effects
@@
 			)
 		)
-		(property "Description" "Resistor, small symbol"
+		(property "Description" "0603WAF0000T5E"
 			(at 33.02 215.9 0)
 			(effects
@@
 			)
 		)
-		(property "Footprint" ""
+		(property "Footprint" "Jumper:SolderJumper-2_P1.3mm_Open_TrianglePad1.0x1.5mm"
 			(at 262.89 95.25 0)
 			(effects
@@
 			)
 		)
-		(property "Footprint" ""
+		(property "Footprint" "Package_SO:PowerIntegrations_SO-8"
 			(at 53.34 208.28 0)
 			(effects
@@
 			)
 		)
-		(property "Footprint" ""
+		(property "Footprint" "Resistor_SMD:R_0603_1608Metric"
 			(at 68.58 215.9 0)
 			(effects
@@
 			)
 		)
-		(property "Description" "Resistor, small symbol"
+		(property "Description" "0603WAF0000T5E"
 			(at 68.58 215.9 0)
 			(effects
@@
 			)
 		)
-		(property "Footprint" ""
+		(property "Footprint" "Jumper:SolderJumper-2_P1.3mm_Open_TrianglePad1.0x1.5mm"
 			(at 231.14 105.41 0)
 			(effects
@@
 			)
 		)
-		(property "Footprint" ""
+		(property "Footprint" "Resistor_SMD:R_0402_1005Metric"
 			(at 199.39 64.77 0)
 			(effects
@@
 			)
 		)
-		(property "Footprint" ""
+		(property "Footprint" "Resistor_SMD:R_0402_1005Metric"
 			(at 151.13 170.18 0)
 			(effects
@@
 			)
 		)
-		(property "Footprint" ""
+		(property "Footprint" "Resistor_SMD:R_0603_1608Metric"
 			(at 33.02 212.09 0)
 			(effects
@@
 			)
 		)
-		(property "Description" "Resistor, small symbol"
+		(property "Description" "0603WAF0000T5E"
 			(at 33.02 212.09 0)
 			(effects
@@
 			)
 		)
-		(property "Footprint" ""
+		(property "Footprint" "Resistor_SMD:R_0402_1005Metric"
 			(at 38.1 269.24 0)
 			(effects
@@
 			)
 		)
-		(property "Footprint" ""
+		(property "Footprint" "Crystal:Crystal_SMD_3215-2Pin_3.2x1.5mm"
 			(at 189.23 71.12 0)
 			(effects
@@
 			)
 		)
-		(property "Datasheet" "~"
+		(property "Datasheet" "https://www.lcsc.com/datasheet/lcsc_datasheet_2210261730_YXC-XKXGI-SUA-32-768K_C5213671.pdf"
 			(at 189.23 71.12 0)
 			(effects
@@
 			)
 		)
-		(property "Description" "Two pin crystal"
+		(property "Description" "XKXGI-SUA-32.768K"
 			(at 189.23 71.12 0)
 			(effects
@@
 			)
 		)
-		(property "Footprint" ""
+		(property "Footprint" "Jumper:SolderJumper-2_P1.3mm_Open_TrianglePad1.0x1.5mm"
 			(at 231.14 115.57 0)
 			(effects
@@
 			)
 		)
-		(property "Footprint" ""
+		(property "Footprint" "Resistor_SMD:R_0402_1005Metric"
 			(at 163.83 105.41 0)
 			(effects
@@
 			)
 		)
-		(property "Footprint" ""
+		(property "Footprint" "Jumper:SolderJumper-2_P1.3mm_Open_TrianglePad1.0x1.5mm"
 			(at 231.14 54.61 0)
 			(effects
@@
 			)
 		)
-		(property "Footprint" ""
+		(property "Footprint" "Jumper:SolderJumper-2_P1.3mm_Open_TrianglePad1.0x1.5mm"
 			(at 231.14 74.93 0)
 			(effects
@@
 			)
 		)
-		(property "Footprint" ""
+		(property "Footprint" "Jumper:SolderJumper-2_P1.3mm_Open_TrianglePad1.0x1.5mm"
 			(at 231.14 69.85 0)
 			(effects
