File: STM32H7B0_devboard/STM32H7B0_devboard.kicad_sch (KiCad schematic)
At the start: 51 parts, among them J2 JTAG, J3 Battery, J4 A, SW1 BTN, SW2 BTN, U1 STM32H7B0VBTx, U7 W25Q128JVS, Y1 25MHz, Y2 32.768 KHz

Commit message: Schematic complete
Parts:
- removed J4: A, symbol Connector_Generic:Conn_01x15
- added J10: I2C1, Connector_PinHeader_2.00mm:PinHeader_1x04_P2.00mm_Vertical, symbol Connector_Generic:Conn_01x04
- added J11: UART1, Connector_PinHeader_2.00mm:PinHeader_1x04_P2.00mm_Vertical, symbol Connector_Generic:Conn_01x04
- added J13: TIM1, Connector_PinHeader_2.00mm:PinHeader_1x06_P2.00mm_Vertical, symbol Connector_Generic:Conn_01x06
- added J15: Power, Connector_PinHeader_2.00mm:PinHeader_2x08_P2.00mm_Vertical, symbol Connector_Generic:Conn_02x08_Counter_Clockwise
- added J4: A, Connector_PinHeader_2.00mm:PinHeader_1x16_P2.00mm_Vertical, symbol Connector_Generic:Conn_01x16
- added J5: B, Connector_PinHeader_2.00mm:PinHeader_1x16_P2.00mm_Vertical, symbol Connector_Generic:Conn_01x16
- added J6: C, Connector_PinHeader_2.00mm:PinHeader_1x16_P2.00mm_Vertical, symbol Connector_Generic:Conn_01x16
- added J7: D, Connector_PinHeader_2.00mm:PinHeader_1x16_P2.00mm_Vertical, symbol Connector_Generic:Conn_01x16
- added J8: E, Connector_PinHeader_2.00mm:PinHeader_1x16_P2.00mm_Vertical, symbol Connector_Generic:Conn_01x16
- added J9: SPI1, Connector_PinHeader_2.00mm:PinHeader_1x06_P2.00mm_Vertical, symbol Connector_Generic:Conn_01x06
- added JP10, JP11, JP12, JP13, JP14, JP15, JP16, JP17, JP18, JP19, JP2, JP20, JP21, JP22, JP23, JP24, JP25, JP26, JP27, JP28, JP3, JP4, JP5, JP6, JP7, JP8, JP9: SolderJumper_2_Open, Jumper:SolderJumper-2_P1.3mm_Open_TrianglePad1.0x1.5mm, symbol Jumper:SolderJumper_2_Open
- added TP1: USB_DP, TestPoint:TestPoint_THTPad_D1.0mm_Drill0.5mm, symbol Connector:TestPoint_Small
- added TP10: QSPI_CLK, TestPoint:TestPoint_THTPad_D1.0mm_Drill0.5mm, symbol Connector:TestPoint_Small
- added TP11: QSPI_IO0, TestPoint:TestPoint_THTPad_D1.0mm_Drill0.5mm, symbol Connector:TestPoint_Small
- added TP12: QSPI_IO1, TestPoint:TestPoint_THTPad_D1.0mm_Drill0.5mm, symbol Connector:TestPoint_Small
- added TP13: QSPI_IO2, TestPoint:TestPoint_THTPad_D1.0mm_Drill0.5mm, symbol Connector:TestPoint_Small
- added TP14: QSPI_IO3, TestPoint:TestPoint_THTPad_D1.0mm_Drill0.5mm, symbol Connector:TestPoint_Small
- added TP2: USB_DN, TestPoint:TestPoint_THTPad_D1.0mm_Drill0.5mm, symbol Connector:TestPoint_Small
- added TP3: HSE_IN, TestPoint:TestPoint_THTPad_D1.0mm_Drill0.5mm, symbol Connector:TestPoint_Small
- added TP4: HSE_OUT, TestPoint:TestPoint_THTPad_D1.0mm_Drill0.5mm, symbol Connector:TestPoint_Small
- added TP5: LSE_IN, TestPoint:TestPoint_THTPad_D1.0mm_Drill0.5mm, symbol Connector:TestPoint_Small
- added TP6: LSE_OUT, TestPoint:TestPoint_THTPad_D1.0mm_Drill0.5mm, symbol Connector:TestPoint_Small
- added TP7: SWCLK, TestPoint:TestPoint_THTPad_D1.0mm_Drill0.5mm, symbol Connector:TestPoint_Small
- added TP8: SWDIO, TestPoint:TestPoint_THTPad_D1.0mm_Drill0.5mm, symbol Connector:TestPoint_Small
- added TP9: QSPI_NCS, TestPoint:TestPoint_THTPad_D1.0mm_Drill0.5mm, symbol Connector:TestPoint_Small
- C1, C2, C3, C4, C5, C6, C7, C8, C9: footprint (none) -> Capacitor_SMD:C_0603_1608Metric
- C11: renamed from C13; footprint (none) -> Capacitor_SMD:C_0603_1608Metric
- D2, D3: footprint (none) -> LED_SMD:LED_0201_0603Metric
- H1, H2, H3, H4: footprint (none) -> MountingHole:MountingHole_3.2mm_M3_Pad_Via
- J2: footprint (none) -> Connector_PinHeader_2.00mm:PinHeader_1x04_P2.00mm_Vertical
- L1: footprint (none) -> Inductor_SMD:L_0805_2012Metric
- R1: renamed from R2; footprint (none) -> Resistor_SMD:R_0603_1608Metric
- R10: renamed from R14; footprint Resistor_SMD:R_0402_1005Metric -> Resistor_SMD:R_0603_1608Metric
- R11: renamed from R15; footprint Resistor_SMD:R_0402_1005Metric -> Resistor_SMD:R_0603_1608Metric
- R2: renamed from R3; footprint (none) -> Resistor_SMD:R_0603_1608Metric
- R3: renamed from R4; footprint (none) -> Resistor_SMD:R_0603_1608Metric
- R4: renamed from R5; footprint (none) -> Resistor_SMD:R_0603_1608Metric
- R5: renamed from R7; footprint (none) -> Resistor_SMD:R_0603_1608Metric
- R6: footprint (none) -> Resistor_SMD:R_0603_1608Metric
- SW1, SW2: footprint (none) -> Button_Switch_SMD:SW_SPST_PTS810
- renumbered C19 to C10, C10 to C13, C11 to C14, D5 to D1, D1 to D4, D4 to D5, R17 to R7, R16 to R8, R18 to R9, U2 to U1, U1 to U2, U7 to U3, U6 to U4
Connections:
- net +3V3: now also J10.1 (Pin_1), J11.1 (Pin_1), J13.1 (Pin_1), J15.13 (Pin_13), J15.14 (Pin_14), J15.15 (Pin_15), J15.16 (Pin_16), J9.1 (Pin_1)
- net +5V: now also J15.10 (Pin_10), J15.11 (Pin_11), J15.12 (Pin_12), J15.9 (Pin_9)
- net GND: now also J10.4 (Pin_4), J11.4 (Pin_4), J13.6 (Pin_6), J15.1 (Pin_1), J15.2 (Pin_2), J15.3 (Pin_3), J15.4 (Pin_4), J15.5 (Pin_5), J15.6 (Pin_6), J15.7 (Pin_7), J15.8 (Pin_8), J9.6 (Pin_6)
- net HSE_IN: now also U2.12 (PH0), TP3.1
- net HSE_OUT: now also U2.13 (PH1), TP4.1
- net LCD_BL: now also JP20.2 (B)
- net LCD_CLK: now also JP17.2 (B)
- net LCD_CMD: now also JP22.2 (B)
- net LCD_MOSI: now also JP19.2 (B)
- net LCD_NCS: now also JP16.2 (B)
- net LCD_NRST: now also JP21.2 (B)
- net LSE_IN: now also U2.8 (PC14), JP2.1 (A), TP5.1
- net LSE_OUT: now also U2.9 (PC15), JP3.1 (A), TP6.1
- net QSPI_CLK: now also JP23.2 (B), TP10.1
- net QSPI_IO0: now also JP25.1 (A), TP11.1
- net QSPI_IO1: now also JP26.1 (A), TP12.1
- net QSPI_IO2: now also JP27.1 (A), TP13.1
- net QSPI_IO3: now also JP28.1 (A), TP14.1
- net QSPI_NCS: now also JP24.2 (B), TP9.1
- net E2: now reaches U2.1 (PE2)
- net E2: now also J8.3 (Pin_3), JP27.2 (B)
- net C0: now reaches U2.15 (PC0)
- net C0: now also J6.1 (Pin_1)
- net C2: now reaches U2.17 (PC2_C)
- net C2: now also J6.3 (Pin_3)
- net C3: now reaches U2.18 (PC3_C)
- net C3: now also J6.4 (Pin_4)
- net E3: now reaches U2.2 (PE3)
- net E3: now also J8.4 (Pin_4)
- net A0: now reaches U2.22 (PA0)
- net A0: now also J4.1 (Pin_1)
- net A1: now reaches U2.23 (PA1)
- net A1: now also J4.2 (Pin_2)
- net A2: now reaches U2.24 (PA2)
- net A2: now also J4.3 (Pin_3), JP20.1 (A)
- net A3: now reaches U2.25 (PA3)
- net A3: now also J4.4 (Pin_4), JP21.1 (A)
- net A4: now reaches U2.28 (PA4)
- net A4: now also J4.5 (Pin_5), JP16.1 (A), JP4.1 (A)
- net A5: now reaches U2.29 (PA5)
- net A5: now also J4.6 (Pin_6), JP17.1 (A), JP5.1 (A)
- net E4: now reaches U2.3 (PE4)
- net E4: now also J8.5 (Pin_5)
- net A6: now reaches U2.30 (PA6)
- net A6: now also J4.7 (Pin_7), JP18.1 (A), JP6.1 (A)
- net A7: now reaches U2.31 (PA7)
- net A7: now also J4.8 (Pin_8), JP19.1 (A), JP7.1 (A)
- net C4: now reaches U2.32 (PC4)
- net C4: now also J6.5 (Pin_5)
- net C5: now reaches U2.33 (PC5)
- net C5: now also J6.6 (Pin_6)
- net B0: now reaches U2.34 (PB0)
- net B0: now also J5.1 (Pin_1)
- net B1: now reaches U2.35 (PB1)
- net B1: now also J5.2 (Pin_2)
- net B2: now reaches U2.36 (PB2)
- net B2: now also J5.3 (Pin_3), JP23.1 (A)
- net E7: now reaches U2.37 (PE7)
- net E7: now also J8.8 (Pin_8)
- net E8: now reaches U2.38 (PE8)
- net E8: now also J8.9 (Pin_9)
- net E9: now reaches U2.39 (PE9)
- net E9: now also J8.10 (Pin_10), JP12.2 (B)
- net E5: now reaches U2.4 (PE5)
- net E5: now also J8.6 (Pin_6)
- net E10: now reaches U2.40 (PE10)
- net E10: now also J8.11 (Pin_11)
- net E11: now reaches U2.41 (PE11)
- net E11: now also J8.12 (Pin_12), JP13.2 (B)
- net E12: now reaches U2.42 (PE12)
- net E12: now also J8.13 (Pin_13)
- net E13: now reaches U2.43 (PE13)
- net E13: now also J8.14 (Pin_14), JP14.2 (B)
- net E14: now reaches U2.44 (PE14)
- net E14: now also J8.15 (Pin_15), JP15.2 (B)
- net E15: now reaches U2.45 (PE15)
- net E15: now also J8.16 (Pin_16)
- net B10: now reaches U2.46 (PB10)
- net B10: now also J5.11 (Pin_11)
- net B11: now reaches U2.47 (PB11)
- net B11: now also J5.12 (Pin_12)
- net E6: now reaches U2.5 (PE6)
- net E6: now also J8.7 (Pin_7)
- net B12: now reaches U2.51 (PB12)
- net B12: now also J5.13 (Pin_13)
- net B13: now reaches U2.52 (PB13)
- net B13: now also J5.14 (Pin_14)
- net B14: now reaches U2.53 (PB14)
- net B14: now also J5.15 (Pin_15)
- net B15: now reaches U2.54 (PB15)
- net B15: now also J5.16 (Pin_16)
- net D8: now reaches U2.55 (PD8)
- net D8: now also J7.9 (Pin_9)
- net D9: now reaches U2.56 (PD9)
- net D9: now also J7.10 (Pin_10)
- net D10: now reaches U2.57 (PD10)
- net D10: now also J7.11 (Pin_11)
- net D11: now reaches U2.58 (PD11)
- net D11: now also J7.12 (Pin_12), JP25.2 (B)
- net D12: now reaches U2.59 (PD12)
- net D12: now also J7.13 (Pin_13), JP26.2 (B)
- net D13: now reaches U2.60 (PD13)
- net D13: now also J7.14 (Pin_14), JP28.2 (B)
- net D14: now reaches U2.61 (PD14)
- net D14: now also J7.15 (Pin_15)
- net D15: now reaches U2.62 (PD15)
- net D15: now also J7.16 (Pin_16)
- net C6: now reaches U2.63 (PC6)
- net C6: now also J6.7 (Pin_7)
- net C7: now reaches U2.64 (PC7)
- net C7: now also J6.8 (Pin_8)
- net C8: now reaches U2.65 (PC8)
- net C8: now also J6.9 (Pin_9)
- net C9: now reaches U2.66 (PC9)
- net C9: now also J6.10 (Pin_10)
- net A8: now reaches U2.67 (PA8)
- net A8: now also J4.9 (Pin_9), JP22.1 (A)
- net A9: now reaches U2.68 (PA9)
- net A9: now also J4.10 (Pin_10), JP8.1 (A)
- net A10: now reaches U2.69 (PA10)
- net A10: now also J4.11 (Pin_11), JP9.1 (A)
- net C13: now reaches U2.7 (PC13)
- net C13: now also J6.14 (Pin_14)
- net A15: now reaches U2.77 (PA15)
- net A15: now also J4.16 (Pin_16)
- net C10: now reaches U2.78 (PC10)
- net C10: now also J6.11 (Pin_11)
- net C11: now reaches U2.79 (PC11)
- net C11: now also J6.12 (Pin_12)
- net C12: now reaches U2.80 (PC12)
- net C12: now also J6.13 (Pin_13)
- net D0: now reaches U2.81 (PD0)
- net D0: now also J7.1 (Pin_1)
- net D1: now reaches U2.82 (PD1)
- net D1: now also J7.2 (Pin_2)
- net D2: now reaches U2.83 (PD2)
- net D2: now also J7.3 (Pin_3)
- net D3: now reaches U2.84 (PD3)
- net D3: now also J7.4 (Pin_4)
- net D4: now reaches U2.85 (PD4)
- net D4: now also J7.5 (Pin_5)
- net D5: now reaches U2.86 (PD5)
- net D5: now also J7.6 (Pin_6)
- net D6: now reaches U2.87 (PD6)
- net D6: now also J7.7 (Pin_7)
- net D7: now reaches U2.88 (PD7)
- net D7: now also J7.8 (Pin_8)
- net B3: now reaches U2.89 (PB3)
- net B3: now also J5.4 (Pin_4)
- net B4: now reaches U2.90 (PB4)
- net B4: now also J5.5 (Pin_5)
- net B5: now reaches U2.91 (PB5)
- net B5: now also J5.6 (Pin_6)
- net B6: now reaches U2.92 (PB6)
- net B6: now also J5.7 (Pin_7), JP24.1 (A)
- net B7: now reaches U2.93 (PB7)
- net B7: now also J5.8 (Pin_8), JP10.1 (A)
- net B8: now reaches U2.95 (PB8)
- net B8: now also J5.9 (Pin_9), JP11.1 (A)
- net B9: now reaches U2.96 (PB9)
- net B9: now also J5.10 (Pin_10)
- net E0: now reaches U2.97 (PE0)
- net E0: now also J8.1 (Pin_1)
- net E1: now reaches U2.98 (PE1)
- net E1: now also J8.2 (Pin_2)
- net STATUS renamed C1
- net C1: now also J6.2 (Pin_2)
- net SWCLK renamed A14
- net A14: now also J4.15 (Pin_15), TP7.1
- net SWDIO renamed A13
- net A13: now also J4.14 (Pin_14), TP8.1
- net USB_DN renamed A11
- net A11: now also J4.12 (Pin_12), TP2.1
- net USB_DP renamed A12
- net A12: now also J4.13 (Pin_13), TP1.1
- new net C14: J6.15 (Pin_15), JP2.2 (B)
- new net C15: J6.16 (Pin_16), JP3.2 (B)
- new net I2C_SCL: J10.2 (Pin_2), JP11.2 (B)
- new net I2C_SDA: J10.3 (Pin_3), JP10.2 (B)
- new net LCD_MISO: JP18.2 (B)
- new net SPI_CLK: J9.3 (Pin_3), JP5.2 (B)
- new net SPI_MISO: J9.4 (Pin_4), JP6.2 (B)
- new net SPI_MOSI: J9.5 (Pin_5), JP7.2 (B)
- new net SPI_NCS: J9.2 (Pin_2), JP4.2 (B)
- new net TIM_CH1: J13.2 (Pin_2), JP12.1 (A)
- new net TIM_CH2: J13.3 (Pin_3), JP13.1 (A)
- new net TIM_CH3: J13.4 (Pin_4), JP14.1 (A)
- new net TIM_CH4: J13.5 (Pin_5), JP15.1 (A)
- new net UART_RX: J11.3 (Pin_3), JP9.2 (B)
- new net UART_TX: J11.2 (Pin_2), JP8.2 (B)
Other:
- sheet LCD ports: added SPI_MISO; removed none
- note added: "LCD connect"
